File: ghlive-hardmod/ghlive-hardmod.kicad_sch (KiCad schematic)
At the start: 14 parts, among them IC1 LDL212D33R, J1 Conn_01x02, J2 Conn_01x02, Q1 Q_PMOS-E_Generic_SGD, Q2 Q_NMOS-E_DGS

Commit message: wip
Parts:
- removed C1: 10nF, PCM_Capacitor_SMD_AKL:C_0603_1608Metric, symbol PCM_Capacitor_AKL:C_Generic
- removed D1, D2: BAT54, Package_TO_SOT_SMD_AKL:SOT-23, symbol PCM_Diode_Schottky_AKL:BAT54
- removed J2: Conn_01x02, symbol Connector_Generic:Conn_01x02
- removed Q1: Q_PMOS-E_Generic_SGD, symbol PCM_Transistor_MOSFET_AKL:Q_PMOS-E_Generic_SGD
- removed Q2: Q_NMOS-E_DGS, symbol PCM_Transistor_MOSFET_AKL:Q_NMOS-E_Generic_DGS
- removed R1: 100K, symbol PCM_Resistor_AKL:R_Generic
- removed R2: 330, symbol PCM_Resistor_AKL:R_Generic
- removed R3: 1M, symbol PCM_Resistor_AKL:R_Generic
- added BOOT1: Conn_01x02, symbol Connector_Generic:Conn_01x02
- added U2: ESP32-S3-WROOM-1, PCM_Espressif:ESP32-S3-WROOM-1, symbol PCM_Espressif:ESP32-S3-WROOM-1
- added UART1: Conn_01x04, symbol Connector_Generic:Conn_01x04
Connections:
- net -BATT: now reaches J1.2 (Pin_2)
- net -BATT: now also C2.1, C3.2, IC1.2 (GND_1), IC1.3 (GND_2), IC1.6 (GND_3), IC1.7 (GND_4), BOOT1.1 (Pin_1), U2.1 (GND), U2.40 (GND), U2.41 (GND), UART1.4 (Pin_4)
- removed net GND: C2.1, C3.2, D3.2 (A), IC1.2 (GND_1), IC1.3 (GND_2), IC1.6 (GND_3), IC1.7 (GND_4), J1.1 (Pin_1)
- net SW_POWER_INPUT renamed +BATT
- net +BATT: now also J1.1 (Pin_1)
- net Vin renamed +3.3V
- net +3.3V: now also U2.2 (3V3), UART1.1 (Pin_1)
- new net: BOOT1.2 (Pin_2), U2.27 (GPIO0/BOOT)
- new net GPIO_POWER_SW: D3.2 (A)
- new net LED_01: U2.28 (SPIIO6/GPIO35/FSPID/SUBSPID)
- new net LED_02: U2.29 (SPIIO7/GPIO36/FSPICLK/SUBSPICLK)
- new net LED_03: U2.13 (GPIO19/U1RTS/ADC2_CH8/CLK_OUT2/USB_D-)
- new net LED_04: U2.14 (GPIO20/U1CTS/ADC2_CH9/CLK_OUT1/USB_D+)
- new net RX: U2.36 (U0RXD/GPIO44/CLK_OUT2), UART1.2 (Pin_2)
- new net SENSE_BATTERY: U2.38 (GPIO2/TOUCH2/ADC1_CH1)
- new net SENSE_WHAMMY: U2.15 (GPIO3/TOUCH3/ADC1_CH2)
- new net SW_B1: U2.18 (GPIO10/TOUCH10/ADC1_CH9/FSPICS0/FSPIIO4/SUBSPICS0)
- new net SW_B2: U2.19 (GPIO11/TOUCH11/ADC2_CH0/FSPID/FSPIIO5/SUBSPID)
- new net SW_B3: U2.21 (GPIO13/TOUCH13/ADC2_CH2/FSPIQ/FSPIIO7/SUBSPIQ)
- new net SW_BT07: U2.11 (GPIO18/U1RXD/ADC2_CH7/CLK_OUT3)
- new net SW_BT08: U2.39 (GPIO1/TOUCH1/ADC1_CH0)
- new net SW_BT09: U2.5 (GPIO5/TOUCH5/ADC1_CH4)
- new net SW_BT10: U2.6 (GPIO6/TOUCH6/ADC1_CH5)
- new net SW_BT11: U2.7 (GPIO7/TOUCH7/ADC1_CH6)
- new net SW_BT12: U2.4 (GPIO4/TOUCH4/ADC1_CH3)
- new net SW_BT13: U2.20 (GPIO12/TOUCH12/ADC2_CH1/FSPICLK/FSPIIO6/SUBSPICLK)
- new net SW_BT14: U2.23 (GPIO21)
- new net SW_BT15: U2.10 (GPIO17/U1TXD/ADC2_CH6)
- new net SW_BT16: U2.8 (GPIO15/U0RTS/ADC2_CH4/XTAL_32K_P)
- new net SW_W1: U2.22 (GPIO14/TOUCH14/ADC2_CH3/FSPIWP/FSPIDQS/SUBSPIWP)
- new net SW_W2: U2.17 (GPIO9/TOUCH9/ADC1_CH8/FSPIHD/SUBSPIHD)
- new net SW_W3: U2.12 (GPIO8/TOUCH8/ADC1_CH7/SUBSPICS1)
- new net TX: U2.37 (U0TXD/GPIO43/CLK_OUT1), UART1.3 (Pin_3)
Other:
- moved on the sheet: C2, C3, D3, IC1

Commit message: Wip schematic
Parts:
- removed BOOT1: Conn_01x02, symbol Connector_Generic:Conn_01x02
- removed UART1: Conn_01x04, symbol Connector_Generic:Conn_01x04
- added C1: C_Generic, symbol PCM_Capacitor_AKL:C_Generic
- added C10: 1uF, symbol PCM_Capacitor_AKL:C_Generic
- added C4, C7, C8, C9: 0.1uF, symbol PCM_Capacitor_AKL:C_Generic
- added C5, C6: 10uF, symbol PCM_Capacitor_AKL:C_Generic
- added D1, D2, D3: ESD9B5.0, symbol PCM_Diode_TVS_AKL:ESD9B5.0
- added D5: D_Generic, symbol PCM_Diode_AKL:D_Generic
- added IC2: SGM2212-3.3XKC3G_TR, symbol SGM2212-3_3XKC3G_TR:SGM2212-3.3XKC3G_TR
- added J2: USB_C_Receptacle_USB2.0_16P, symbol Connector:USB_C_Receptacle_USB2.0_16P
- added J3: Conn_01x07_Socket, symbol Connector:Conn_01x07_Socket
- added LED1: LED, symbol Device:LED
- added Q2: Q_PNP_Generic_BCE, symbol PCM_Transistor_BJT_AKL:Q_PNP_Generic_BCE
- added R1, R2, R3: 5.1k, symbol PCM_Resistor_AKL:R_Generic
- added R4, R5: 10k, symbol PCM_Resistor_AKL:R_Generic
- added SW1, SW2: SW_MEC_5E, symbol Switch:SW_MEC_5E
- IC1: footprint SOIC127P600X175-8N -> (none)
- U2: footprint PCM_Espressif:ESP32-S3-WROOM-1 -> (none)
- renumbered D3 to D4
Connections:
- net +3.3V: now also C6.2, C7.1, IC2.2 (VOUT_1), IC2.4 (VOUT_2), R3.2, R4.2, R5.2
- net GPIO_POWER_HOLD: now also D5.2 (A); no longer D4.1 (K), IC1.5 (EN)
- net LED_03: now also U2.16 (GPIO46); no longer U2.13 (GPIO19/U1RTS/ADC2_CH8/CLK_OUT2/USB_D-)
- net LED_04: now also U2.26 (GPIO45); no longer U2.14 (GPIO20/U1CTS/ADC2_CH9/CLK_OUT1/USB_D+)
- net SW_B1: now also J3.4 (Pin_4)
- net SW_B2: now also J3.3 (Pin_3)
- net SW_B3: now also J3.2 (Pin_2)
- net SW_W1: now also J3.1 (Pin_1)
- net SW_W2: now also J3.5 (Pin_5)
- net SW_W3: now also J3.6 (Pin_6)
- net at U2.27 (GPIO0/BOOT): now also C8.1, SW1.1, SW1.2
- net at U2.3 (EN): now also C10.1, C9.1, R4.1, SW2.1, SW2.2
- net -BATT renamed GND
- net GND: now also C1.2, C10.2, C4.2, C5.1, C6.1, C7.2, C8.2, C9.2, IC2.1 (GND), J2.A1 (GND), J2.A12 (GND), J2.B1 (GND), J2.B12 (GND), J2.S1 (SHIELD), J3.7 (Pin_7), LED1.1 (K), R1.1, R2.1, SW1.3 (K), SW1.4 (A), SW2.3 (K), SW2.4 (A)
- net RX: no longer names the net of U2.36 (U0RXD/GPIO44/CLK_OUT2)
- net TX: no longer names the net of U2.37 (U0TXD/GPIO43/CLK_OUT1)
- new net: IC1.5 (EN), Q2.2 (C)
- new net: C1.1, D1.1 (K), D2.1 (K), D3.1 (K)
- new net: D4.1 (K), D5.1 (K), Q2.3 (E)
- new net: J2.A5 (CC1), R2.2
- new net: Q2.1 (B), R5.1
- new net: J2.B5 (CC2), R1.2
- new net: LED1.2 (A), R3.1
- new net +5V: C4.1, C5.2, D3.2 (A), IC2.3 (VIN), J2.A4 (VBUS), J2.A9 (VBUS), J2.B4 (VBUS), J2.B9 (VBUS)
- new net USB_D+: D2.2 (A), J2.A6 (D+), J2.B6 (D+), U2.14 (GPIO20/U1CTS/ADC2_CH9/CLK_OUT1/USB_D+)
- new net USB_D-: D1.2 (A), J2.A7 (D-), J2.B7 (D-), U2.13 (GPIO19/U1RTS/ADC2_CH8/CLK_OUT2/USB_D-)
- no-connect marks 0 -> 4
Other:
- moved on the sheet: D4, J1, U2

Commit message: wip
Parts:
- added D6: D_Generic, symbol PCM_Diode_AKL:D_Generic
Connections:
- net +3.3V: now also D6.2 (A); no longer R5.2
- new net: D6.1 (K), R5.2
Other:
- moved on the sheet: R5
Changed lines of the file:
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@@
 	)
 	(junction
-		(at 80.01 60.96)
+		(at 80.01 71.12)
 		(diameter 0)
 		(color 0 0 0 0)
 	)
 	(junction
-		(at 80.01 71.12)
+		(at 86.36 116.84)
 		(diameter 0)
 		(color 0 0 0 0)
 	)
 	(junction
-		(at 86.36 116.84)
+		(at 57.15 130.81)
 		(diameter 0)
 		(color 0 0 0 0)
 	)
 	(junction
-		(at 57.15 130.81)
+		(at 80.01 67.31)
 		(diameter 0)
 		(color 0 0 0 0)
@@
 	(wire
 		(pts
-			(xy 46.99 31.75) (xy 82.55 31.75)
+			(xy 82.55 67.31) (xy 80.01 67.31)
 		)
 		(stroke
@@
 	(wire
 		(pts
-			(xy 106.68 55.88) (xy 109.22 55.88)
+			(xy 46.99 31.75) (xy 82.55 31.75)
 		)
 		(stroke
@@
 	(wire
 		(pts
-			(xy 240.03 101.6) (xy 242.57 101.6)
+			(xy 106.68 55.88) (xy 109.22 55.88)
 		)
 		(stroke
@@
 	(wire
 		(pts
-			(xy 86.36 154.94) (xy 90.17 154.94)
+			(xy 240.03 101.6) (xy 242.57 101.6)
 		)
 		(stroke
@@
 	(wire
 		(pts
-			(xy 82.55 39.37) (xy 82.55 40.64)
+			(xy 86.36 154.94) (xy 90.17 154.94)
 		)
 		(stroke
@@
 	(wire
 		(pts
-			(xy 68.58 116.84) (xy 68.58 118.11)
+			(xy 82.55 39.37) (xy 82.55 40.64)
 		)
 		(stroke
@@
 	(wire
 		(pts
-			(xy 91.44 60.96) (xy 90.17 60.96)
+			(xy 68.58 116.84) (xy 68.58 118.11)
 		)
 		(stroke
@@
 	(wire
 		(pts
+			(xy 91.44 67.31) (xy 91.44 66.04)
+		)
+		(stroke
+			(width 0)
+			(type default)
+		)
+	)
+	(wire
+		(pts
+			(xy 80.01 67.31) (xy 80.01 71.12)
+		)
+		(stroke
+			(width 0)
+			(type default)
+		)
+	)
+	(wire
+		(pts
 			(xy 240.03 129.54) (xy 242.57 129.54)
 		)
@@
 	(wire
 		(pts
+			(xy 80.01 71.12) (xy 82.55 71.12)
+		)
+		(stroke
+			(width 0)
+			(type default)
+		)
+	)
+	(wire
+		(pts
 			(xy 46.99 31.75) (xy 46.99 35.56)
 		)
@@
 	(wire
 		(pts
-			(xy 80.01 71.12) (xy 82.55 71.12)
-		)
-		(stroke
-			(width 0)
-			(type default)
-		)
-	)
-	(wire
-		(pts
 			(xy 60.96 133.35) (xy 76.2 133.35)
 		)
@@
 	(wire
 		(pts
+			(xy 90.17 67.31) (xy 91.44 67.31)
+		)
+		(stroke
+			(width 0)
+			(type default)
+		)
+	)
+	(wire
+		(pts
 			(xy 275.59 91.44) (xy 275.59 93.98)
 		)
@@
 	(wire
 		(pts
+			(xy 77.47 60.96) (xy 77.47 67.31)
+		)
+		(stroke
+			(width 0)
+			(type default)
+		)
+	)
+	(wire
+		(pts
 			(xy 240.03 78.74) (xy 242.57 78.74)
 		)
@@
 	(wire
 		(pts
-			(xy 80.01 60.96) (xy 82.55 60.96)
-		)
-		(stroke
-			(width 0)
-			(type default)
-		)
-	)
-	(wire
-		(pts
-			(xy 91.44 58.42) (xy 91.44 60.96)
-		)
-		(stroke
-			(width 0)
-			(type default)
-		)
-	)
-	(wire
-		(pts
 			(xy 82.55 39.37) (xy 95.25 39.37)
 		)
@@
 	(wire
 		(pts
-			(xy 80.01 60.96) (xy 80.01 71.12)
+			(xy 102.87 16.51) (xy 99.06 16.51)
 		)
 		(stroke
@@
 	(wire
 		(pts
-			(xy 102.87 16.51) (xy 99.06 16.51)
+			(xy 146.05 78.74) (xy 148.59 78.74)
 		)
 		(stroke
@@
 	(wire
 		(pts
-			(xy 146.05 78.74) (xy 148.59 78.74)
+			(xy 34.29 60.96) (xy 77.47 60.96)
 		)
 		(stroke
@@
 	(wire
 		(pts
-			(xy 34.29 60.96) (xy 80.01 60.96)
+			(xy 57.15 116.84) (xy 59.69 116.84)
 		)
 		(stroke
@@
 	(wire
 		(pts
-			(xy 57.15 116.84) (xy 59.69 116.84)
+			(xy 106.68 45.72) (xy 109.22 45.72)
 		)
 		(stroke
@@
 	(wire
 		(pts
-			(xy 106.68 45.72) (xy 109.22 45.72)
+			(xy 76.2 111.76) (xy 71.12 111.76)
 		)
 		(stroke
@@
 	(wire
 		(pts
-			(xy 76.2 111.76) (xy 71.12 111.76)
+			(xy 80.01 67.31) (xy 77.47 67.31)
 		)
 		(stroke
@@
 	)
 	(symbol
+		(lib_id "PCM_Diode_AKL:D_Generic")
+		(at 86.36 67.31 0)
+		(unit 1)
+		(exclude_from_sim no)
+		(in_bom yes)
+		(on_board yes)
+		(dnp no)
+		(property "Reference" "D6"
+			(at 84.328 61.722 0)
+			(effects
+				(font
+					(size 1.27 1.27)
+				)
+			)
+		)
+		(property "Value" "D_Generic"
+			(at 84.836 64.262 0)
+			(effects
+				(font
+					(size 1.27 1.27)
+				)
+			)
+		)
+		(property "Footprint" ""
+			(at 86.36 67.31 0)
+			(effects
+				(font
+					(size 1.27 1.27)
+				)
+				(hide yes)
+			)
+		)
+		(property "Datasheet" "~"
+			(at 86.36 67.31 0)
+			(effects
+				(font
+					(size 1.27 1.27)
+				)
+				(hide yes)
+			)
+		)
+		(property "Description" "Diode, Generic symbol, Alternate KiCad Library"
+			(at 86.36 67.31 0)
+			(effects
+				(font
+					(size 1.27 1.27)
+				)
+				(hide yes)
+			)
+		)
+		(pin "1"
+		)
+		(pin "2"
+		)
+		(instances
+			(project "ghlive-hardmod"
+				(path "/e4d12dac-785e-45c9-8b5d-9ae68fcce16f"
+					(reference "D6")
+					(unit 1)
+				)
+			)
+		)
+	)
+	(symbol
 		(lib_id "PCM_Resistor_AKL:R_Generic")
 		(at 63.5 116.84 270)
@@
 	(symbol
 		(lib_id "PCM_Resistor_AKL:R_Generic")
-		(at 86.36 60.96 270)
+		(at 91.44 62.23 0)
 		(unit 1)
 		(exclude_from_sim no)
@@
 		(dnp no)
 		(property "Reference" "R5"
-			(at 86.36 60.96 90)
+			(at 91.44 62.23 90)
 			(effects
 				(font
@@
 		)
 		(property "Value" "10k"
-			(at 86.36 63.246 90)
+			(at 93.726 62.23 90)
 			(effects
 				(font
@@
 		)
 		(property "Footprint" ""
-			(at 86.36 59.182 90)
+			(at 89.662 62.23 90)
 			(effects
 				(font
@@
 		)
 		(property "Datasheet" "~"
-			(at 86.36 60.96 0)
+			(at 91.44 62.23 0)
 			(effects
 				(font
@@
 		)
 		(property "Description" "Resistor, Generic European Symbol, Alternate KiCad Library"
-			(at 86.36 60.96 0)
+			(at 91.44 62.23 0)
 			(effects
 				(font
